File: dsPIC33-schematic.kicad_pcb (KiCad board)
At the start: 2 copper layers, 36.8 x 71.1 mm, 15 parts, among them IC1 DSPIC33EP64MC502-I_SP, IC2 LM2937ET-3.3_NOPB, J1 Conn_01x05_Male, J2 Conn_01x16_Female, J3 Conn_01x10_Male, J4 Conn_01x03_Male, J5 Conn_01x01, J6 Conn_01x01

Commit message: added PCB layout and gerber files
Other:
- board text added: "@sharmavins23"
- board text added: "dsPIC33 LCD Controller"
- board text removed: "5V"
- board text removed: "GND"
Changed lines of the file:
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@@
     (visible_elements FFFDEF7F)
     (pcbplotparams
-      (layerselection 0x010fc_ffffffff)
+      (layerselection 0x010f0_ffffffff)
       (usegerberextensions false)
       (usegerberattributes true)
@@
       (outputformat 1)
       (mirror false)
-      (drillshape 1)
+      (drillshape 0)
       (scaleselection 1)
       (outputdirectory ""))
@@
       (net 2 GND))
   )
-  (gr_text GND (at 157.48 66.04) (layer F.Cu)
-    (effects (font (size 1.5 1.5) (thickness 0.3)))
-  )
-  (gr_text 5V (at 127 66.04) (layer F.Cu)
-    (effects (font (size 1.5 1.5) (thickness 0.3)))
+  (gr_text "dsPIC33 LCD Controller" (at 135.89 64.77) (layer F.SilkS)
+    (effects (font (size 1 1) (thickness 0.15)))
+  )
+  (gr_text @sharmavins23 (at 132.08 133.35) (layer F.SilkS)
+    (effects (font (size 1 1) (thickness 0.15)))
   )
   (gr_arc (start 149.86 123.19) (end 161.29 123.19) (angle 90) (layer Edge.Cuts) (width 0.05))
